Commit message: new file:   description/lidar.xacro 	modified:   description/robot.urdf.xacro 	modified:   description/robot_core.xacro

File: description/robot.urdf.xacro (robot description, xacro)
@@ -5,3 +5,4 @@
     <xacro:include filename="inertial_macros.xacro"/>
     <xacro:include filename="gazebo_control.xacro" />
+    <xacro:include filename="lidar.xacro"/>
 </robot>

File: description/robot_core.xacro (robot description, xacro)
@@ -13,4 +13,7 @@
     <material name="black">
         <color rgba="0 0 0 1"/>
+    </material>
+    <material name="red">
+        <color rgba="1 0 0 1"/>
     </material>
     <!--BASE LINK-->
