Commit message: corrected robot_structure and camera setup

File: description/camera.xacro (robot description, xacro)
@@ -40,5 +40,5 @@
         <parent link="camera_link"/>
         <child link="camera_link_optical"/>
-        <origin xyz="0 0 0" rpy="${-3.14/2} 0 ${3.14/2}"/>
+        <origin xyz="0 0 0" rpy="-1.5708 0 1.5708"/>
     </joint>
     <link name="camera_link_optical">

File: description/depth_camera.xacro (robot description, xacro)
@@ -16,5 +16,5 @@
     <gazebo reference="depth_camera_link">
         <material>Gazebo/Green</material>
-        <sensor name="camera" type="depth">
+        <sensor name="depth_camera" type="depth">
             <pose>0 0 0 0 0 0</pose>
             <visualize>true</visualize>
@@ -33,7 +33,10 @@
             </camera>
             <plugin name="depth_camera_controller" filename="libgazebo_ros_camera.so">
-                <min_depth>0.1</min_depth>
-                <max_depth>5</max_depth>
-                <frame_name>camera_link_optical</frame_name>
+                <camera_name>depth_camera</camera_name>
+                <frame_name>depth_camera_link_optical</frame_name>
+                <image_topic_name>image_raw</image_topic_name>
+                <camera_info_topic_name>camera_info</camera_info_topic_name>
+                <depth_image_topic_name>depth/image_raw</depth_image_topic_name>
+                <depth_camera_info_topic_name>depth/camera_info</depth_camera_info_topic_name>
             </plugin>
         </sensor>
@@ -42,5 +45,5 @@
         <parent link="depth_camera_link"/>
         <child link="depth_camera_link_optical"/>
-        <origin xyz="0 0 0" rpy="${3.14/2} ${3.14/2} 0"/>
+        <origin xyz="0 0 0" rpy="-1.5708 0 1.5708"/>
     </joint>
     <link name="depth_camera_link_optical">

File: description/gazebo_control.xacro (robot description, xacro)
@@ -20,8 +20,3 @@
         </plugin>
     </gazebo>
-    <gazebo>
-        <plugin name="model_state_publisher" filename="libgazebo_ros_state.so">
-            <update_rate>30</update_rate>
-        </plugin>
-    </gazebo>
 </robot>

File: description/robot.urdf.xacro (robot description, xacro)
@@ -9,4 +9,4 @@
     <xacro:include filename="camera.xacro"/>
     <xacro:include filename="gazebo_model.xacro"/>
-    <!--<xacro:include filename="depth_camera.xacro"/>-->
+    <!-- <xacro:include filename="depth_camera.xacro"/> -->
 </robot>

File: description/robot_structure.xacro (robot description, xacro)
@@ -30,5 +30,5 @@
         <child link="round_body"/>
         <!--origin at center of base_link, with 5 cm ground clearance-->
-        <origin xyz="0 0 0.05"/>
+        <origin xyz="0 0 0.05" rpy="0 0 0"/>
     </joint>
     <link name="round_body">
@@ -57,5 +57,5 @@
         <parent link="base_link"/>
         <child link="left_wheel"/>
-        <origin xyz="-0.15 0.25 0" rpy="${-3.14/2} 0 0"/>
+        <origin xyz="0.15 0.25 0" rpy="${-3.14/2} 0 0"/>
         <axis xyz="0 0 1"/>
     </joint>
@@ -83,5 +83,5 @@
         <parent link="base_link"/>
         <child link="right_wheel"/>
-        <origin xyz="-0.15 -0.25 0" rpy="${3.14/2} 0 0"/>
+        <origin xyz="0.15 -0.25 0" rpy="${3.14/2} 0 0"/>
         <axis xyz="0 0 -1"/>
     </joint>
