Commit message: added depth camera

File: .history/description/depth_camera_20240917091837.xacro (robot description, xacro)
@@ -4,5 +4,5 @@
         <parent link="round_body"/>
         <child link="camera_link"/>
-        <origin xyz="0.3 0 0.02" rpy="0 0 0"/>
+        <origin xyz="0.3 0 0.05" rpy="0 0 0"/>
     </joint>
     <link name="camera_link">

File: .history/description/depth_camera_20240917092020.xacro (robot description, xacro)
@@ -4,5 +4,5 @@
         <parent link="round_body"/>
         <child link="camera_link"/>
-        <origin xyz="0.3 0 0.02" rpy="0 0 0"/>
+        <origin xyz="0.3 0 0.05" rpy="0 0 0"/>
     </joint>
     <link name="camera_link">
@@ -16,5 +16,5 @@
     <gazebo reference="camera_link">
         <material>Gazebo/Green</material>
-        <sensor name="camera" type="camera">
+        <sensor name="camera" type="depth">
             <pose>0 0 0 0 0 0</pose>
             <visualize>true</visualize>

File: .history/description/depth_camera_20240917093101.xacro (robot description, xacro)
@@ -4,5 +4,5 @@
         <parent link="round_body"/>
         <child link="camera_link"/>
-        <origin xyz="0.3 0 0.02" rpy="0 0 0"/>
+        <origin xyz="0.3 0 0.05" rpy="0 0 0"/>
     </joint>
     <link name="camera_link">
@@ -16,5 +16,5 @@
     <gazebo reference="camera_link">
         <material>Gazebo/Green</material>
-        <sensor name="camera" type="camera">
+        <sensor name="camera" type="depth">
             <pose>0 0 0 0 0 0</pose>
             <visualize>true</visualize>
@@ -40,5 +40,5 @@
         <parent link="camera_link"/>
         <child link="camera_link_optical"/>
-        <origin xyz="0 0 0" rpy="${-3.14/2} 0 ${3.14/2}"/>
+        <origin xyz="0 0 0" rpy="${3.14/2} 0 ${3.14/2}"/>
     </joint>
     <link name="camera_link_optical">

File: .history/description/depth_camera_20240917093532.xacro (robot description, xacro)
@@ -4,5 +4,5 @@
         <parent link="round_body"/>
         <child link="camera_link"/>
-        <origin xyz="0.3 0 0.02" rpy="0 0 0"/>
+        <origin xyz="0.3 0 0.05" rpy="0 0 0"/>
     </joint>
     <link name="camera_link">
@@ -16,5 +16,5 @@
     <gazebo reference="camera_link">
         <material>Gazebo/Green</material>
-        <sensor name="camera" type="camera">
+        <sensor name="camera" type="depth">
             <pose>0 0 0 0 0 0</pose>
             <visualize>true</visualize>
@@ -40,5 +40,5 @@
         <parent link="camera_link"/>
         <child link="camera_link_optical"/>
-        <origin xyz="0 0 0" rpy="${-3.14/2} 0 ${3.14/2}"/>
+        <origin xyz="0 0 0" rpy="${3.14/2} ${3.14/2}"/>
     </joint>
     <link name="camera_link_optical">

File: .history/description/depth_camera_20240917093534.xacro (robot description, xacro)
@@ -4,5 +4,5 @@
         <parent link="round_body"/>
         <child link="camera_link"/>
-        <origin xyz="0.3 0 0.02" rpy="0 0 0"/>
+        <origin xyz="0.3 0 0.05" rpy="0 0 0"/>
     </joint>
     <link name="camera_link">
@@ -16,5 +16,5 @@
     <gazebo reference="camera_link">
         <material>Gazebo/Green</material>
-        <sensor name="camera" type="camera">
+        <sensor name="camera" type="depth">
             <pose>0 0 0 0 0 0</pose>
             <visualize>true</visualize>
@@ -40,5 +40,5 @@
         <parent link="camera_link"/>
         <child link="camera_link_optical"/>
-        <origin xyz="0 0 0" rpy="${-3.14/2} 0 ${3.14/2}"/>
+        <origin xyz="0 0 0" rpy="${3.14/2} ${3.14/2} 0"/>
     </joint>
     <link name="camera_link_optical">

File: .history/description/depth_camera_20240917093725.xacro (robot description, xacro)
@@ -4,5 +4,5 @@
         <parent link="round_body"/>
         <child link="camera_link"/>
-        <origin xyz="0.3 0 0.02" rpy="0 0 0"/>
+        <origin xyz="0.3 0 0.05" rpy="0 0 0"/>
     </joint>
     <link name="camera_link">
@@ -16,5 +16,5 @@
     <gazebo reference="camera_link">
         <material>Gazebo/Green</material>
-        <sensor name="camera" type="camera">
+        <sensor name="camera" type="depth">
             <pose>0 0 0 0 0 0</pose>
             <visualize>true</visualize>
@@ -40,5 +40,5 @@
         <parent link="camera_link"/>
         <child link="camera_link_optical"/>
-        <origin xyz="0 0 0" rpy="${-3.14/2} 0 ${3.14/2}"/>
+        <origin xyz="0 0 0" rpy="${3.14/2} 0 ${3.14/2} 0"/>
     </joint>
     <link name="camera_link_optical">

File: .history/description/depth_camera_20240917093727.xacro (robot description, xacro)
@@ -4,5 +4,5 @@
         <parent link="round_body"/>
         <child link="camera_link"/>
-        <origin xyz="0.3 0 0.02" rpy="0 0 0"/>
+        <origin xyz="0.3 0 0.05" rpy="0 0 0"/>
     </joint>
     <link name="camera_link">
@@ -16,5 +16,5 @@
     <gazebo reference="camera_link">
         <material>Gazebo/Green</material>
-        <sensor name="camera" type="camera">
+        <sensor name="camera" type="depth">
             <pose>0 0 0 0 0 0</pose>
             <visualize>true</visualize>
@@ -40,5 +40,5 @@
         <parent link="camera_link"/>
         <child link="camera_link_optical"/>
-        <origin xyz="0 0 0" rpy="${-3.14/2} 0 ${3.14/2}"/>
+        <origin xyz="0 0 0" rpy="${3.14/2} 0 ${-3.14/2} 0"/>
     </joint>
     <link name="camera_link_optical">

File: .history/description/depth_camera_20240917093729.xacro (robot description, xacro)
@@ -4,5 +4,5 @@
         <parent link="round_body"/>
         <child link="camera_link"/>
-        <origin xyz="0.3 0 0.02" rpy="0 0 0"/>
+        <origin xyz="0.3 0 0.05" rpy="0 0 0"/>
     </joint>
     <link name="camera_link">
@@ -16,5 +16,5 @@
     <gazebo reference="camera_link">
         <material>Gazebo/Green</material>
-        <sensor name="camera" type="camera">
+        <sensor name="camera" type="depth">
             <pose>0 0 0 0 0 0</pose>
             <visualize>true</visualize>
@@ -40,5 +40,5 @@
         <parent link="camera_link"/>
         <child link="camera_link_optical"/>
-        <origin xyz="0 0 0" rpy="${-3.14/2} 0 ${3.14/2}"/>
+        <origin xyz="0 0 0" rpy="${3.14/2} 0 ${-3.14/2}/>
     </joint>
     <link name="camera_link_optical">

File: .history/description/depth_camera_20240917093730.xacro (robot description, xacro)
@@ -4,5 +4,5 @@
         <parent link="round_body"/>
         <child link="camera_link"/>
-        <origin xyz="0.3 0 0.02" rpy="0 0 0"/>
+        <origin xyz="0.3 0 0.05" rpy="0 0 0"/>
     </joint>
     <link name="camera_link">
@@ -16,5 +16,5 @@
     <gazebo reference="camera_link">
         <material>Gazebo/Green</material>
-        <sensor name="camera" type="camera">
+        <sensor name="camera" type="depth">
             <pose>0 0 0 0 0 0</pose>
             <visualize>true</visualize>
@@ -40,5 +40,5 @@
         <parent link="camera_link"/>
         <child link="camera_link_optical"/>
-        <origin xyz="0 0 0" rpy="${-3.14/2} 0 ${3.14/2}"/>
+        <origin xyz="0 0 0" rpy="${3.14/2} 0 ${-3.14/2}"/>
     </joint>
     <link name="camera_link_optical">

File: .history/description/depth_camera_20240917094110.xacro (robot description, xacro)
@@ -4,5 +4,5 @@
         <parent link="round_body"/>
         <child link="camera_link"/>
-        <origin xyz="0.3 0 0.02" rpy="0 0 0"/>
+        <origin xyz="0.3 0 0.05" rpy="0 0 0"/>
     </joint>
     <link name="camera_link">
@@ -16,5 +16,5 @@
     <gazebo reference="camera_link">
         <material>Gazebo/Green</material>
-        <sensor name="camera" type="camera">
+        <sensor name="camera" type="depth">
             <pose>0 0 0 0 0 0</pose>
             <visualize>true</visualize>
@@ -40,5 +40,5 @@
         <parent link="camera_link"/>
         <child link="camera_link_optical"/>
-        <origin xyz="0 0 0" rpy="${-3.14/2} 0 ${3.14/2}"/>
+        <origin xyz="0 0 0" rpy="${-3.14/2} 0 ${-3.14/2}"/>
     </joint>
     <link name="camera_link_optical">

File: .history/description/depth_camera_20240917094845.xacro (robot description, xacro)
@@ -4,5 +4,5 @@
         <parent link="round_body"/>
         <child link="camera_link"/>
-        <origin xyz="0.3 0 0.02" rpy="0 0 0"/>
+        <origin xyz="0.3 0 0.06" rpy="0 0 0"/>
     </joint>
     <link name="camera_link">
@@ -16,5 +16,5 @@
     <gazebo reference="camera_link">
         <material>Gazebo/Green</material>
-        <sensor name="camera" type="camera">
+        <sensor name="camera" type="depth">
             <pose>0 0 0 0 0 0</pose>
             <visualize>true</visualize>
@@ -40,5 +40,5 @@
         <parent link="camera_link"/>
         <child link="camera_link_optical"/>
-        <origin xyz="0 0 0" rpy="${-3.14/2} 0 ${3.14/2}"/>
+        <origin xyz="0 0 0" rpy="${-3.14/2} 0 ${-3.14/2}"/>
     </joint>
     <link name="camera_link_optical">

File: .history/description/depth_camera_20240917095015.xacro (robot description, xacro)
@@ -3,6 +3,6 @@
     <joint name="camera_joint" type="fixed">
         <parent link="round_body"/>
-        <child link="camera_link"/>
-        <origin xyz="0.3 0 0.02" rpy="0 0 0"/>
+        <child link="depthcamera_link"/>
+        <origin xyz="0.3 0 0.06" rpy="0 0 0"/>
     </joint>
     <link name="camera_link">
@@ -16,5 +16,5 @@
     <gazebo reference="camera_link">
         <material>Gazebo/Green</material>
-        <sensor name="camera" type="camera">
+        <sensor name="camera" type="depth">
             <pose>0 0 0 0 0 0</pose>
             <visualize>true</visualize>
@@ -40,5 +40,5 @@
         <parent link="camera_link"/>
         <child link="camera_link_optical"/>
-        <origin xyz="0 0 0" rpy="${-3.14/2} 0 ${3.14/2}"/>
+        <origin xyz="0 0 0" rpy="${-3.14/2} 0 ${-3.14/2}"/>
     </joint>
     <link name="camera_link_optical">

File: .history/description/depth_camera_20240917095016.xacro (robot description, xacro)
@@ -3,6 +3,6 @@
     <joint name="camera_joint" type="fixed">
         <parent link="round_body"/>
-        <child link="camera_link"/>
-        <origin xyz="0.3 0 0.02" rpy="0 0 0"/>
+        <child link="depth_camera_link"/>
+        <origin xyz="0.3 0 0.06" rpy="0 0 0"/>
     </joint>
     <link name="camera_link">
@@ -16,5 +16,5 @@
     <gazebo reference="camera_link">
         <material>Gazebo/Green</material>
-        <sensor name="camera" type="camera">
+        <sensor name="camera" type="depth">
             <pose>0 0 0 0 0 0</pose>
             <visualize>true</visualize>
@@ -40,5 +40,5 @@
         <parent link="camera_link"/>
         <child link="camera_link_optical"/>
-        <origin xyz="0 0 0" rpy="${-3.14/2} 0 ${3.14/2}"/>
+        <origin xyz="0 0 0" rpy="${-3.14/2} 0 ${-3.14/2}"/>
     </joint>
     <link name="camera_link_optical">

File: .history/description/depth_camera_20240917095026.xacro (robot description, xacro)
@@ -3,6 +3,6 @@
     <joint name="camera_joint" type="fixed">
         <parent link="round_body"/>
-        <child link="camera_link"/>
-        <origin xyz="0.3 0 0.02" rpy="0 0 0"/>
+        <child link="depth_camera_link"/>
+        <origin xyz="0.3 0 0.06" rpy="0 0 0"/>
     </joint>
     <link name="camera_link">
@@ -16,5 +16,5 @@
     <gazebo reference="camera_link">
         <material>Gazebo/Green</material>
-        <sensor name="camera" type="camera">
+        <sensor name="camera" type="depth">
             <pose>0 0 0 0 0 0</pose>
             <visualize>true</visualize>
@@ -38,7 +38,7 @@
     </gazebo>
     <joint name="camera_optical_joint" type="fixed">
-        <parent link="camera_link"/>
+        <parent link="depth_camera_link"/>
         <child link="camera_link_optical"/>
-        <origin xyz="0 0 0" rpy="${-3.14/2} 0 ${3.14/2}"/>
+        <origin xyz="0 0 0" rpy="${-3.14/2} 0 ${-3.14/2}"/>
     </joint>
     <link name="camera_link_optical">

File: .history/description/depth_camera_20240917095048.xacro (robot description, xacro)
@@ -3,6 +3,6 @@
     <joint name="camera_joint" type="fixed">
         <parent link="round_body"/>
-        <child link="camera_link"/>
-        <origin xyz="0.3 0 0.02" rpy="0 0 0"/>
+        <child link="depth_camera_link"/>
+        <origin xyz="0.3 0 0.06" rpy="0 0 0"/>
     </joint>
     <link name="camera_link">
@@ -16,5 +16,5 @@
     <gazebo reference="camera_link">
         <material>Gazebo/Green</material>
-        <sensor name="camera" type="camera">
+        <sensor name="camera" type="depth">
             <pose>0 0 0 0 0 0</pose>
             <visualize>true</visualize>
@@ -38,7 +38,7 @@
     </gazebo>
     <joint name="camera_optical_joint" type="fixed">
-        <parent link="camera_link"/>
-        <child link="camera_link_optical"/>
-        <origin xyz="0 0 0" rpy="${-3.14/2} 0 ${3.14/2}"/>
+        <parent link="depth_camera_link"/>
+        <child link="depth_camera_link_optical"/>
+        <origin xyz="0 0 0" rpy="${-3.14/2} 0 ${-3.14/2}"/>
     </joint>
     <link name="camera_link_optical">

File: .history/description/depth_camera_20240917095051.xacro (robot description, xacro)
@@ -3,6 +3,6 @@
     <joint name="camera_joint" type="fixed">
         <parent link="round_body"/>
-        <child link="camera_link"/>
-        <origin xyz="0.3 0 0.02" rpy="0 0 0"/>
+        <child link="depth_camera_link"/>
+        <origin xyz="0.3 0 0.06" rpy="0 0 0"/>
     </joint>
     <link name="camera_link">
@@ -16,5 +16,5 @@
     <gazebo reference="camera_link">
         <material>Gazebo/Green</material>
-        <sensor name="camera" type="camera">
+        <sensor name="camera" type="depth">
             <pose>0 0 0 0 0 0</pose>
             <visualize>true</visualize>
@@ -38,9 +38,9 @@
     </gazebo>
     <joint name="camera_optical_joint" type="fixed">
-        <parent link="camera_link"/>
-        <child link="camera_link_optical"/>
-        <origin xyz="0 0 0" rpy="${-3.14/2} 0 ${3.14/2}"/>
+        <parent link="depth_camera_link"/>
+        <child link="depth_camera_link_optical"/>
+        <origin xyz="0 0 0" rpy="${-3.14/2} 0 ${-3.14/2}"/>
     </joint>
-    <link name="camera_link_optical">
+    <link name="depthcamera_link_optical">
     </link>
 </robot>

File: .history/description/depth_camera_20240917095052.xacro (robot description, xacro)
@@ -3,6 +3,6 @@
     <joint name="camera_joint" type="fixed">
         <parent link="round_body"/>
-        <child link="camera_link"/>
-        <origin xyz="0.3 0 0.02" rpy="0 0 0"/>
+        <child link="depth_camera_link"/>
+        <origin xyz="0.3 0 0.06" rpy="0 0 0"/>
     </joint>
     <link name="camera_link">
@@ -16,5 +16,5 @@
     <gazebo reference="camera_link">
         <material>Gazebo/Green</material>
-        <sensor name="camera" type="camera">
+        <sensor name="camera" type="depth">
             <pose>0 0 0 0 0 0</pose>
             <visualize>true</visualize>
@@ -38,9 +38,9 @@
     </gazebo>
     <joint name="camera_optical_joint" type="fixed">
-        <parent link="camera_link"/>
-        <child link="camera_link_optical"/>
-        <origin xyz="0 0 0" rpy="${-3.14/2} 0 ${3.14/2}"/>
+        <parent link="depth_camera_link"/>
+        <child link="depth_camera_link_optical"/>
+        <origin xyz="0 0 0" rpy="${-3.14/2} 0 ${-3.14/2}"/>
     </joint>
-    <link name="camera_link_optical">
+    <link name="depth_camera_link_optical">
     </link>
 </robot>

File: .history/description/depth_camera_20240917095105.xacro (robot description, xacro)
@@ -3,6 +3,6 @@
     <joint name="camera_joint" type="fixed">
         <parent link="round_body"/>
-        <child link="camera_link"/>
-        <origin xyz="0.3 0 0.02" rpy="0 0 0"/>
+        <child link="depth_camera_link"/>
+        <origin xyz="0.3 0 0.06" rpy="0 0 0"/>
     </joint>
     <link name="camera_link">
@@ -16,5 +16,5 @@
     <gazebo reference="camera_link">
         <material>Gazebo/Green</material>
-        <sensor name="camera" type="camera">
+        <sensor name="camera" type="depth">
             <pose>0 0 0 0 0 0</pose>
             <visualize>true</visualize>
@@ -37,10 +37,10 @@
         </sensor>
     </gazebo>
-    <joint name="camera_optical_joint" type="fixed">
-        <parent link="camera_link"/>
-        <child link="camera_link_optical"/>
-        <origin xyz="0 0 0" rpy="${-3.14/2} 0 ${3.14/2}"/>
+    <joint name="depth_camera_optical_joint" type="fixed">
+        <parent link="depth_camera_link"/>
+        <child link="depth_camera_link_optical"/>
+        <origin xyz="0 0 0" rpy="${-3.14/2} 0 ${-3.14/2}"/>
     </joint>
-    <link name="camera_link_optical">
+    <link name="depth_camera_link_optical">
     </link>
 </robot>

File: .history/description/depth_camera_20240917095113.xacro (robot description, xacro)
@@ -3,6 +3,6 @@
     <joint name="camera_joint" type="fixed">
         <parent link="round_body"/>
-        <child link="camera_link"/>
-        <origin xyz="0.3 0 0.02" rpy="0 0 0"/>
+        <child link="depth_camera_link"/>
+        <origin xyz="0.3 0 0.06" rpy="0 0 0"/>
     </joint>
     <link name="camera_link">
@@ -14,7 +14,7 @@
         </visual>
     </link>
-    <gazebo reference="camera_link">
+    <gazebo reference="depth_camera_link">
         <material>Gazebo/Green</material>
-        <sensor name="camera" type="camera">
+        <sensor name="camera" type="depth">
             <pose>0 0 0 0 0 0</pose>
             <visualize>true</visualize>
@@ -37,10 +37,10 @@
         </sensor>
     </gazebo>
-    <joint name="camera_optical_joint" type="fixed">
-        <parent link="camera_link"/>
-        <child link="camera_link_optical"/>
-        <origin xyz="0 0 0" rpy="${-3.14/2} 0 ${3.14/2}"/>
+    <joint name="depth_camera_optical_joint" type="fixed">
+        <parent link="depth_camera_link"/>
+        <child link="depth_camera_link_optical"/>
+        <origin xyz="0 0 0" rpy="${-3.14/2} 0 ${-3.14/2}"/>
     </joint>
-    <link name="camera_link_optical">
+    <link name="depth_camera_link_optical">
     </link>
 </robot>

File: .history/description/depth_camera_20240917095117.xacro (robot description, xacro)
@@ -3,8 +3,8 @@
     <joint name="camera_joint" type="fixed">
         <parent link="round_body"/>
-        <child link="camera_link"/>
-        <origin xyz="0.3 0 0.02" rpy="0 0 0"/>
+        <child link="depth_camera_link"/>
+        <origin xyz="0.3 0 0.06" rpy="0 0 0"/>
     </joint>
-    <link name="camera_link">
+    <link name="depth_camera_link">
         <visual>
             <geometry>
@@ -14,7 +14,7 @@
         </visual>
     </link>
-    <gazebo reference="camera_link">
+    <gazebo reference="depth_camera_link">
         <material>Gazebo/Green</material>
-        <sensor name="camera" type="camera">
+        <sensor name="camera" type="depth">
             <pose>0 0 0 0 0 0</pose>
             <visualize>true</visualize>
@@ -37,10 +37,10 @@
         </sensor>
     </gazebo>
-    <joint name="camera_optical_joint" type="fixed">
-        <parent link="camera_link"/>
-        <child link="camera_link_optical"/>
-        <origin xyz="0 0 0" rpy="${-3.14/2} 0 ${3.14/2}"/>
+    <joint name="depth_camera_optical_joint" type="fixed">
+        <parent link="depth_camera_link"/>
+        <child link="depth_camera_link_optical"/>
+        <origin xyz="0 0 0" rpy="${-3.14/2} 0 ${-3.14/2}"/>
     </joint>
-    <link name="camera_link_optical">
+    <link name="depth_camera_link_optical">
     </link>
 </robot>
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